File: controller/pcb/piPDU.kicad_pcb (KiCad board)
At the start: 2 copper layers, 36 parts, among them J35 Raspberry_Pi_2_3

Commit message: Fix PCB and schematic redundant connections
Parts:
- removed BTN1: SCR_BTN1, TerminalBlock:TerminalBlock_bornier-2_P5.08mm
- removed BTN10: SCR_BTN10, TerminalBlock:TerminalBlock_bornier-2_P5.08mm
- removed BTN11: SCR_BTN11, TerminalBlock:TerminalBlock_bornier-2_P5.08mm
- removed BTN12: SCR_BTN12, TerminalBlock:TerminalBlock_bornier-2_P5.08mm
- removed BTN13: SCR_BTN13, TerminalBlock:TerminalBlock_bornier-2_P5.08mm
- removed BTN14: SCR_BTN14, TerminalBlock:TerminalBlock_bornier-2_P5.08mm
- removed BTN15: SCR_BTN15, TerminalBlock:TerminalBlock_bornier-2_P5.08mm
- removed BTN16: SCR_BTN16, TerminalBlock:TerminalBlock_bornier-2_P5.08mm
- removed BTN2: SCR_BTN2, TerminalBlock:TerminalBlock_bornier-2_P5.08mm
- removed BTN3: SCR_BTN3, TerminalBlock:TerminalBlock_bornier-2_P5.08mm
- removed BTN4: SCR_BTN4, TerminalBlock:TerminalBlock_bornier-2_P5.08mm
- removed BTN5: SCR_BTN5, TerminalBlock:TerminalBlock_bornier-2_P5.08mm
- removed BTN6: SCR_BTN6, TerminalBlock:TerminalBlock_bornier-2_P5.08mm
- removed BTN7: SCR_BTN7, TerminalBlock:TerminalBlock_bornier-2_P5.08mm
- removed BTN8: SCR_BTN8, TerminalBlock:TerminalBlock_bornier-2_P5.08mm
- removed BTN9: SCR_BTN9, TerminalBlock:TerminalBlock_bornier-2_P5.08mm
- removed LCD_COM: SCR_LCD_DATA, TerminalBlock:TerminalBlock_bornier-2_P5.08mm
- removed LCD_POW: SCR_LCD_PWR, TerminalBlock:TerminalBlock_bornier-2_P5.08mm
- removed LED1: SCR_LED1, TerminalBlock:TerminalBlock_bornier-2_P5.08mm
- removed LED10: SCR_LED10, TerminalBlock:TerminalBlock_bornier-2_P5.08mm
- removed LED11: SCR_LED11, TerminalBlock:TerminalBlock_bornier-2_P5.08mm
- removed LED12: SCR_LED12, TerminalBlock:TerminalBlock_bornier-2_P5.08mm
- removed LED13: SCR_LED13, TerminalBlock:TerminalBlock_bornier-2_P5.08mm
- removed LED14: SCR_LED14, TerminalBlock:TerminalBlock_bornier-2_P5.08mm
- removed LED15: SCR_LED15, TerminalBlock:TerminalBlock_bornier-2_P5.08mm
- removed LED16: SCR_LED16, TerminalBlock:TerminalBlock_bornier-2_P5.08mm
- removed LED2: SCR_LED2, TerminalBlock:TerminalBlock_bornier-2_P5.08mm
- removed LED3: SCR_LED3, TerminalBlock:TerminalBlock_bornier-2_P5.08mm
- removed LED4: SCR_LED4, TerminalBlock:TerminalBlock_bornier-2_P5.08mm
- removed LED5: SCR_LED5, TerminalBlock:TerminalBlock_bornier-2_P5.08mm
- removed LED6: SCR_LED6, TerminalBlock:TerminalBlock_bornier-2_P5.08mm
- removed LED7: SCR_LED7, TerminalBlock:TerminalBlock_bornier-2_P5.08mm
- removed LED8: SCR_LED8, TerminalBlock:TerminalBlock_bornier-2_P5.08mm
- removed LED9: SCR_LED9, TerminalBlock:TerminalBlock_bornier-2_P5.08mm
- removed POWER_IN: SCR_5V, TerminalBlock:TerminalBlock_bornier-2_P5.08mm
- added J0: SCR_BTN1, TerminalBlock:TerminalBlock_bornier-2_P5.08mm, F.Cu at (30.5, 27.9)
- added J1: SCR_LED1, TerminalBlock:TerminalBlock_bornier-2_P5.08mm, F.Cu at (30.5, 48.3)
- added J10: SCR_BTN6, TerminalBlock:TerminalBlock_bornier-2_P5.08mm, F.Cu at (106.7, 27.4)
- added J11: SCR_LED6, TerminalBlock:TerminalBlock_bornier-2_P5.08mm, F.Cu at (106.7, 48.3)
- added J12: SCR_BTN7, TerminalBlock:TerminalBlock_bornier-2_P5.08mm, F.Cu at (121.9, 27.2)
- added J13: SCR_LED7, TerminalBlock:TerminalBlock_bornier-2_P5.08mm, F.Cu at (121.9, 48.3)
- added J14: SCR_BTN8, TerminalBlock:TerminalBlock_bornier-2_P5.08mm, F.Cu at (137.2, 27.2)
- added J15: SCR_LED8, TerminalBlock:TerminalBlock_bornier-2_P5.08mm, F.Cu at (137.2, 48.3)
- added J16: SCR_BTN9, TerminalBlock:TerminalBlock_bornier-2_P5.08mm, F.Cu at (152.4, 27.2)
- added J17: SCR_LED9, TerminalBlock:TerminalBlock_bornier-2_P5.08mm, F.Cu at (152.4, 48.0)
- added J18: SCR_BTN10, TerminalBlock:TerminalBlock_bornier-2_P5.08mm, F.Cu at (167.6, 27.2)
- added J19: SCR_LED10, TerminalBlock:TerminalBlock_bornier-2_P5.08mm, F.Cu at (167.6, 48.0)
- added J2: SCR_BTN2, TerminalBlock:TerminalBlock_bornier-2_P5.08mm, F.Cu at (45.7, 27.7)
- added J20: SCR_BTN11, TerminalBlock:TerminalBlock_bornier-2_P5.08mm, F.Cu at (182.9, 27.2)
- added J21: SCR_LED11, TerminalBlock:TerminalBlock_bornier-2_P5.08mm, F.Cu at (182.9, 48.0)
- added J22: SCR_BTN12, TerminalBlock:TerminalBlock_bornier-2_P5.08mm, F.Cu at (198.1, 27.2)
- added J23: SCR_LED12, TerminalBlock:TerminalBlock_bornier-2_P5.08mm, F.Cu at (198.1, 48.0)
- added J24: SCR_BTN13, TerminalBlock:TerminalBlock_bornier-2_P5.08mm, F.Cu at (213.4, 27.2)
- added J25: SCR_LED13, TerminalBlock:TerminalBlock_bornier-2_P5.08mm, F.Cu at (213.4, 48.0)
- added J26: SCR_BTN14, TerminalBlock:TerminalBlock_bornier-2_P5.08mm, F.Cu at (228.6, 27.2)
- added J27: SCR_LED14, TerminalBlock:TerminalBlock_bornier-2_P5.08mm, F.Cu at (228.6, 48.0)
- added J28: SCR_BTN15, TerminalBlock:TerminalBlock_bornier-2_P5.08mm, F.Cu at (243.8, 27.2)
- added J29: SCR_LED15, TerminalBlock:TerminalBlock_bornier-2_P5.08mm, F.Cu at (243.8, 48.0)
- added J3: SCR_LED2, TerminalBlock:TerminalBlock_bornier-2_P5.08mm, F.Cu at (45.7, 48.3)
- added J30: SCR_BTN16, TerminalBlock:TerminalBlock_bornier-2_P5.08mm, F.Cu at (259.1, 26.9)
- added J31: SCR_LED16, TerminalBlock:TerminalBlock_bornier-2_P5.08mm, F.Cu at (259.1, 48.0)
- added J32: SCR_5V, TerminalBlock:TerminalBlock_bornier-2_P5.08mm, F.Cu at (30.2, 99.1)
- added J33: SCR_LCD_PWR, TerminalBlock:TerminalBlock_bornier-2_P5.08mm, F.Cu at (261.6, 94.0)
- added J34: SCR_LCD_DATA, TerminalBlock:TerminalBlock_bornier-2_P5.08mm, F.Cu at (261.6, 78.7)
- added J4: SCR_BTN3, TerminalBlock:TerminalBlock_bornier-2_P5.08mm, F.Cu at (61.0, 27.7)
- added J5: SCR_LED3, TerminalBlock:TerminalBlock_bornier-2_P5.08mm, F.Cu at (61.0, 48.3)
- added J6: SCR_BTN4, TerminalBlock:TerminalBlock_bornier-2_P5.08mm, F.Cu at (76.2, 27.7)
- added J7: SCR_LED4, TerminalBlock:TerminalBlock_bornier-2_P5.08mm, F.Cu at (76.2, 48.3)
- added J8: SCR_BTN5, TerminalBlock:TerminalBlock_bornier-2_P5.08mm, F.Cu at (91.4, 27.4)
- added J9: SCR_LED5, TerminalBlock:TerminalBlock_bornier-2_P5.08mm, F.Cu at (91.4, 48.3)
Connections:
- J35 pad 1: +3V3 -> unconnected-(J35-Pad1)
- J35 pad 17: +3V3 -> unconnected-(J35-Pad17)
- J35 pad 20: GND -> unconnected-(J35-Pad20)
- J35 pad 25: GND -> unconnected-(J35-Pad25)
- J35 pad 30: GND -> unconnected-(J35-Pad30)
- J35 pad 34: GND -> unconnected-(J35-Pad34)
- J35 pad 39: GND -> unconnected-(J35-Pad39)
- J35 pad 4: +5V -> unconnected-(J35-Pad4)
- J35 pad 6: GND -> unconnected-(J35-Pad6)
Routing:
- net GND: track 705.2 -> 756.1 mm

Commit message: Add board outline
Other:
- board outline added: 251.5 x 117.9 mm
Changed lines of the file:
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@@
     )
   )
+  (gr_rect (start 271.78 7.62) (end 20.32 125.476) (layer "Edge.Cuts") (width 0.1) (fill none))
   (gr_text "-  +" (at 124.46 40.64) (layer "F.SilkS")
     (effects (font (size 1.5 1.5) (thickness 0.3)))

Commit message: Add mounting holes to PCB
Parts:
- moved J1 23.6 mm to (30.5, 71.9)
- moved J11 23.6 mm to (106.7, 71.9)
- moved J13 23.6 mm to (121.9, 71.9)
- moved J15 23.6 mm to (137.2, 71.9)
- moved J3 23.6 mm to (45.7, 71.9)
- moved J5 23.6 mm to (61.0, 71.9)
- moved J7 23.6 mm to (76.2, 71.9)
- moved J9 23.6 mm to (91.4, 71.9)
- moved J10 23.6 mm to (106.7, 51.1)
- moved J8 23.6 mm to (91.4, 51.1)
- moved J17 23.6 mm to (152.4, 71.6)
- moved J19 23.6 mm to (167.6, 71.6)
- moved J2 23.6 mm to (45.7, 51.3)
- moved J21 23.6 mm to (182.9, 71.6)
- moved J23 23.6 mm to (198.1, 71.6)
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Routing:
- net GND: track 756.1 -> 762.6 mm
- net Net-(J34-Pad1): track 114.5 -> 117.9 mm
- net Net-(J34-Pad2): track 118.5 -> 121.9 mm
- net row8: track 142.8 -> 140.5 mm
Other:
- outline, holes or cut-outs redrawn

Commit message: Save project
Other:
- board text added: "PI PDU CONTROLLER BOARD REV 1.1 AUTHOR: MIRCEA ANTON"
- board text removed: "PI PDU CONTROLLER BOARD REV 1.0 AUTHOR: MIRCEA ANTON"
Changed lines of the file:
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@@
     (effects (font (size 1.5 1.5) (thickness 0.3)))
   )
-  (gr_text "PI PDU CONTROLLER BOARD\nREV 1.0\nAUTHOR: MIRCEA ANTON" (at 58.42 120.142) (layer "F.SilkS")
+  (gr_text "PI PDU CONTROLLER BOARD\nREV 1.1\nAUTHOR: MIRCEA ANTON" (at 58.42 120.142) (layer "F.SilkS")
     (effects (font (size 1.5 1.5) (thickness 0.3)))
   )

Commit message: Update PCB design for DIY printing
Parts:
- moved J30 0.46 mm to (259.0, 51.0)
Routing:
- net row1: track 474.1 -> 422.5 mm, vias 0 -> 2
- net row2: track 402.8 -> 369.7 mm, vias 0 -> 2
- net row3: track 344.4 -> 314.9 mm, vias 0 -> 2
- net row4: track 285.9 -> 258.7 mm, vias 0 -> 2
- net row5: track 263.5 -> 240.0 mm, vias 0 -> 2
- net col2: track 355.1 -> 333.2 mm, vias 0 -> 2
- net row6: track 221.8 -> 200.5 mm, vias 0 -> 2
- net row7: track 184.3 -> 165.6 mm, vias 0 -> 2
- net col1: track 292.0 -> 281.3 mm, vias 0 -> 2
- net row8: track 140.5 -> 133.0 mm, vias 0 -> 2

Commit message: Make tracks thicker and more spaced out
Connections:
- J35 pad 9: GND -> unconnected-(J35-Pad9)
Routing:
- net GND: track 762.6 -> 579.4 mm
- net col1: track 281.3 -> 433.1 mm
- net row5: track 240.0 -> 359.9 mm
- net col2: track 333.2 -> 426.2 mm
- net row6: track 200.5 -> 290.0 mm
- net row1: track 422.5 -> 502.3 mm
- net +5V: track 389.8 -> 311.9 mm, vias 0 -> 3
- net row7: track 165.6 -> 235.3 mm, vias 2 -> 3
- net row2: track 369.7 -> 429.1 mm, vias 2 -> 3
- net row3: track 314.9 -> 367.3 mm, vias 2 -> 3
- net row4: track 258.7 -> 306.8 mm, vias 2 -> 3
- net row8: track 133.0 -> 178.2 mm
- net LED3: track 89.9 -> 105.5 mm
- net LED10: track 63.0 -> 76.4 mm
- net LED2: track 103.2 -> 115.9 mm
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Other:
- board size 251.5 x 117.9 mm -> 251.5 x 119.9 mm
- board text removed: "- +"

Commit message: Update controller PCB and schematic to use GPIO expanders
Parts:
- removed J17: SCR_LED9, TerminalBlock:TerminalBlock_bornier-2_P5.08mm
- removed J18: SCR_BTN10, TerminalBlock:TerminalBlock_bornier-2_P5.08mm
- removed J19: SCR_LED10, TerminalBlock:TerminalBlock_bornier-2_P5.08mm
- removed J20: SCR_BTN11, TerminalBlock:TerminalBlock_bornier-2_P5.08mm
- removed J21: SCR_LED11, TerminalBlock:TerminalBlock_bornier-2_P5.08mm
- removed J22: SCR_BTN12, TerminalBlock:TerminalBlock_bornier-2_P5.08mm
- removed J23: SCR_LED12, TerminalBlock:TerminalBlock_bornier-2_P5.08mm
- removed J24: SCR_BTN13, TerminalBlock:TerminalBlock_bornier-2_P5.08mm
- removed J25: SCR_LED13, TerminalBlock:TerminalBlock_bornier-2_P5.08mm
- removed J26: SCR_BTN14, TerminalBlock:TerminalBlock_bornier-2_P5.08mm
- removed J27: SCR_LED14, TerminalBlock:TerminalBlock_bornier-2_P5.08mm
- removed J28: SCR_BTN15, TerminalBlock:TerminalBlock_bornier-2_P5.08mm
- removed J29: SCR_LED15, TerminalBlock:TerminalBlock_bornier-2_P5.08mm
- removed J30: SCR_BTN16, TerminalBlock:TerminalBlock_bornier-2_P5.08mm
- removed J31: SCR_LED16, TerminalBlock:TerminalBlock_bornier-2_P5.08mm
- removed J32: SCR_5V, TerminalBlock:TerminalBlock_bornier-2_P5.08mm
- removed J33: SCR_LCD_PWR, TerminalBlock:TerminalBlock_bornier-2_P5.08mm
- removed J34: SCR_LCD_DATA, TerminalBlock:TerminalBlock_bornier-2_P5.08mm
- removed J35: Raspberry_Pi_2_3, Module:Raspberry_Pi_Zero_Socketed_THT_FaceDown_MountingHoles
- added U5: 8P_Header, Connector_PinHeader_2.54mm:PinHeader_1x08_P2.54mm_Vertical, F.Cu at (35.6, 44.1)
- added U6: 8P_Header, Connector_PinHeader_2.54mm:PinHeader_1x08_P2.54mm_Vertical, F.Cu at (88.1, 43.9)
- added U7: 8P_Header, Connector_PinHeader_2.54mm:PinHeader_1x08_P2.54mm_Vertical, F.Cu at (193.0, 43.9)
- added U8: 8P_Header, Connector_PinHeader_2.54mm:PinHeader_1x08_P2.54mm_Vertical, F.Cu at (140.6, 43.9)
- J0: value SCR_BTN1 -> SCR_5V
- J1: value SCR_LED1 -> SCR_BTN_1; footprint TerminalBlock:TerminalBlock_bornier-2_P5.08mm -> TerminalBlock:TerminalBlock_bornier-3_P5.08mm
- J10: value SCR_BTN6 -> SCR_BTN_10; footprint TerminalBlock:TerminalBlock_bornier-2_P5.08mm -> TerminalBlock:TerminalBlock_bornier-3_P5.08mm
- J11: value SCR_LED6 -> SCR_BTN_11; footprint TerminalBlock:TerminalBlock_bornier-2_P5.08mm -> TerminalBlock:TerminalBlock_bornier-3_P5.08mm
- J12: value SCR_BTN7 -> SCR_BTN_12; footprint TerminalBlock:TerminalBlock_bornier-2_P5.08mm -> TerminalBlock:TerminalBlock_bornier-3_P5.08mm
- J13: value SCR_LED7 -> SCR_BTN_13; footprint TerminalBlock:TerminalBlock_bornier-2_P5.08mm -> TerminalBlock:TerminalBlock_bornier-3_P5.08mm
- J14: value SCR_BTN8 -> SCR_BTN_14; footprint TerminalBlock:TerminalBlock_bornier-2_P5.08mm -> TerminalBlock:TerminalBlock_bornier-3_P5.08mm
- J15: value SCR_LED8 -> SCR_BTN_15; footprint TerminalBlock:TerminalBlock_bornier-2_P5.08mm -> TerminalBlock:TerminalBlock_bornier-3_P5.08mm
- J16: value SCR_BTN9 -> SCR_BTN_16; footprint TerminalBlock:TerminalBlock_bornier-2_P5.08mm -> TerminalBlock:TerminalBlock_bornier-3_P5.08mm
- J2: value SCR_BTN2 -> SCR_BTN_2; footprint TerminalBlock:TerminalBlock_bornier-2_P5.08mm -> TerminalBlock:TerminalBlock_bornier-3_P5.08mm
- J3: value SCR_LED2 -> SCR_BTN_3; footprint TerminalBlock:TerminalBlock_bornier-2_P5.08mm -> TerminalBlock:TerminalBlock_bornier-3_P5.08mm
- J4: value SCR_BTN3 -> SCR_BTN_4; footprint TerminalBlock:TerminalBlock_bornier-2_P5.08mm -> TerminalBlock:TerminalBlock_bornier-3_P5.08mm
- J5: value SCR_LED3 -> SCR_BTN_5; footprint TerminalBlock:TerminalBlock_bornier-2_P5.08mm -> TerminalBlock:TerminalBlock_bornier-3_P5.08mm
- J6: value SCR_BTN4 -> SCR_BTN_6; footprint TerminalBlock:TerminalBlock_bornier-2_P5.08mm -> TerminalBlock:TerminalBlock_bornier-3_P5.08mm
- J7: value SCR_LED4 -> SCR_BTN_7; footprint TerminalBlock:TerminalBlock_bornier-2_P5.08mm -> TerminalBlock:TerminalBlock_bornier-3_P5.08mm
- J8: value SCR_BTN5 -> SCR_BTN_8; footprint TerminalBlock:TerminalBlock_bornier-2_P5.08mm -> TerminalBlock:TerminalBlock_bornier-3_P5.08mm
- J9: value SCR_LED5 -> SCR_BTN_9; footprint TerminalBlock:TerminalBlock_bornier-2_P5.08mm -> TerminalBlock:TerminalBlock_bornier-3_P5.08mm
- moved J0 207.7 mm to (237.5, 34.1), turned to 90 degrees
- moved J8 124.3 mm to (212.1, 21.1)
- moved J7 117.0 mm to (181.6, 21.1)
- moved J6 88.7 mm to (159.6, 21.1)
- moved J5 85.0 mm to (129.1, 21.1)
- moved J9 77.3 mm to (24.1, 33.9)
- moved J16 62.1 mm to (212.1, 33.8)
- moved J3 59.5 mm to (76.6, 21.1)
- moved J15 58.5 mm to (181.6, 33.8)
- moved J4 55.2 mm to (107.1, 21.1)
- moved J10 54.8 mm to (54.6, 33.9)
- moved J1 51.1 mm to (24.1, 21.2)
- moved J11 48.5 mm to (76.6, 33.8)
- moved J13 38.8 mm to (129.1, 33.8)
- moved J2 31.4 mm to (54.6, 21.2)
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Connections:
- J0 pad 1: row1 -> GND
- J0 pad 2: col2 -> +5V
- J1 pad 1: GND -> LED1
- J1 pad 2: LED1 -> +5V
- J10 pad 1: row6 -> LED10
- J10 pad 2: col2 -> +5V
- J11 pad 1: GND -> LED11
- J11 pad 2: LED6 -> +5V
- J12 pad 1: row7 -> LED12
- J12 pad 2: col2 -> +5V
- J13 pad 1: GND -> LED13
- J13 pad 2: LED7 -> +5V
- J14 pad 1: row8 -> LED14
- J14 pad 2: col2 -> +5V
- J15 pad 1: GND -> LED15
- J15 pad 2: LED8 -> +5V
- J16 pad 1: row8 -> LED16
- J16 pad 2: col1 -> +5V
- J2 pad 1: row2 -> LED2
- J2 pad 2: col2 -> +5V
- J3 pad 1: GND -> LED3
- J3 pad 2: LED2 -> +5V
- J4 pad 1: row3 -> LED4
- J4 pad 2: col2 -> +5V
- J5 pad 1: GND -> LED5
- J5 pad 2: LED3 -> +5V
- J6 pad 1: row4 -> LED6
- J6 pad 2: col2 -> +5V
- J7 pad 1: GND -> LED7
- J7 pad 2: LED4 -> +5V
- J8 pad 1: row5 -> LED8
- J8 pad 2: col2 -> +5V
- J9 pad 1: GND -> LED9
- J9 pad 2: LED5 -> +5V
Routing:
- net GND: track 579.4 -> 0.00 mm
- net row1: track 502.3 -> 0.00 mm, vias 2 -> 0
- net col1: track 433.1 -> 0.00 mm, vias 2 -> 0
- net row2: track 429.1 -> 0.00 mm, vias 3 -> 0
- net col2: track 426.2 -> 0.00 mm, vias 2 -> 0
- net row3: track 367.3 -> 0.00 mm, vias 3 -> 0
- net row5: track 359.9 -> 0.00 mm, vias 2 -> 0
- net row4: track 306.8 -> 0.00 mm, vias 3 -> 0
- net row6: track 290.0 -> 0.00 mm, vias 2 -> 0
- net row7: track 235.3 -> 0.00 mm, vias 3 -> 0
- net row8: track 178.2 -> 0.00 mm, vias 2 -> 0
- net Net-(J34-Pad2): track 123.5 -> 0.00 mm
- net Net-(J34-Pad1): track 119.6 -> 0.00 mm
- net LED16: track 129.0 -> 16.5 mm
- net LED1: track 135.8 -> 41.9 mm
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Other:
- board outline removed
- board text removed: "5V"
- board text removed: "GND"
- board text removed: "PI PDU CONTROLLER BOARD REV 1.1 AUTHOR: MIRCEA ANTON"
- board text removed: "PI ZERO"
- board text removed: "SCL"
- board text removed: "SDA"

Commit message: Update controller pcb and schematic to use GPIO expanders
Parts:
- added J17: SCR_5V2, TerminalBlock:TerminalBlock_bornier-2_P5.08mm, F.Cu at (242.6, 30.9)
- added J18: SCR_i2c, TerminalBlock:TerminalBlock_bornier-2_P5.08mm, F.Cu at (268.0, 38.9)
- added J19: SCR_i2c, TerminalBlock:TerminalBlock_bornier-2_P5.08mm, F.Cu at (268.0, 26.2)
- added J20: SCR_i2c, TerminalBlock:TerminalBlock_bornier-2_P5.08mm, F.Cu at (268.0, 51.6)
- J0: value SCR_5V -> SCR_5V1
- moved J0 219.7 mm to (17.8, 30.9)
- moved J12 8.70 mm to (114.7, 38.0)
- moved J13 8.70 mm to (136.7, 38.0)
- moved J14 8.70 mm to (167.2, 38.0)
- moved J15 8.70 mm to (189.2, 38.0)
- moved J16 8.70 mm to (219.7, 38.0)
- moved J4 8.70 mm to (114.7, 25.3)
- moved J5 8.70 mm to (136.7, 25.3)
- moved J6 8.70 mm to (167.2, 25.3)
- moved J7 8.70 mm to (189.2, 25.3)
- moved J8 8.70 mm to (219.7, 25.3)
- moved U6 8.70 mm to (95.7, 48.1)
- moved U7 8.70 mm to (200.7, 48.1)
- moved J1 8.70 mm to (31.8, 25.4)
- moved J9 8.70 mm to (31.8, 38.1)
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Routing:
- net GND: track 0.00 -> 275.6 mm
- net +5V: track 363.9 -> 441.5 mm
- net SDA: track 0.00 -> 52.3 mm
- net SCL: track 0.00 -> 44.4 mm
